File: chess-board-iot.kicad_sch (KiCad schematic)
At the start: 19 parts

Commit message: update main schematic with hierarchical sheets
Parts:
- removed D?: (no value), symbol Device:D_Schottky_Small
- added C101: (no value), symbol Device:C_Small
- added H101, H102, H103, H104, H105, H106, H107, H108, H109: (no value), symbol Mechanical:MountingHole
- added OLED101, OLED102, OLED103: (no value), symbol User_Symbols:OLED_I2C
- added R101, R105, R106, R107, R108, R111, R112: (no value), symbol Device:R_Small
- added SW101, SW102, SW103, SW104, SW105, SW106, SW107, SW108, SW109: (no value), symbol Switch:SW_SPST
- added U104: (no value), symbol Interface_Expansion:PCA9548APW
- C102: renamed from C?; value 22uF -> (none); footprint Capacitor_SMD:C_0603_1608Metric -> (none)
- C103: renamed from C?; value 4.7uF -> (none); footprint Capacitor_SMD:C_0805_2012Metric -> (none); LCSC C1779 -> C19666
- C104: renamed from C?; LCSC (none) -> C53987
- C105: renamed from C?; LCSC (none) -> C14663
- C106: renamed from C?; value 100nF -> (none); LCSC (none) -> C14663
- Q101, Q102: renamed from Q?; symbol Transistor_BJT:S8050 -> Transistor_BJT:MMBTA42; LCSC (none) -> C2146
- R104: renamed from R?; LCSC C17514 -> C22935
- R109: renamed from R?; footprint Resistor_SMD:R_0805_2012Metric -> (none); LCSC C17514 -> C25804
- R110: renamed from R?; value 10K -> (none); footprint Resistor_SMD:R_0805_2012Metric -> (none); LCSC C17514 -> C25804
- U101: renamed from U?; value XC6220B331MR-G -> (none); footprint Package_TO_SOT_SMD:SOT-23-5 -> (none)
- U103: renamed from U?; LCSC (none) -> C85364
- gave numbers to parts that had none: 6
Connections:
- net 3V3: now also C106.1, U102.2 (VDD), U105.6 (VDD), OLED101.2 (VCC), OLED102.2 (VCC), OLED103.2 (VCC), R101.1, R105.1, R106.1, R107.2, R108.2, R111.1, R112.2, U104.24 (VCC)
- net DTR: now also Q102.2 (E); no longer Q102.1 (E)
- net EN: now also U102.3 (EN), C101.1, R101.2
- net GND: now also U102.1 (GND), U102.15 (GND), U102.38 (GND), U102.39 (GND), C101.2, OLED101.1 (GND), OLED102.1 (GND), OLED103.1 (GND), SW101.2 (B), SW102.2 (B), SW103.2 (B), SW104.2 (B), SW105.2 (B), SW106.2 (B), SW107.2 (B), SW108.2 (B), SW109.2 (B), U104.12 (GND)
- net IO0: now also U102.25 (IO0)
- net RTS: now also Q101.2 (E); no longer Q101.1 (E)
- net RXD: now also U102.35 (TXD0/IO1)
- net TXD: now also U102.34 (RXD0/IO3)
- net VBUS: now also J101.A4 (VBUS), J101.A9 (VBUS), J101.B4 (VBUS), J101.B9 (VBUS), U103.5 (VP), U105.7 (VREGIN); no longer C106.1
- net at R110.1: now also Q102.1 (B); no longer Q102.2 (B)
- net I2C_A0: now reaches U102.10 (IO25)
- net I2C_A0: now also U104.1 (A0)
- net I2C_A1: now reaches U102.11 (IO26)
- net I2C_A1: now also U104.2 (A1)
- net I2C_A2: now reaches U102.12 (IO27)
- net I2C_A2: now also U104.21 (A2)
- net ~{IO_INT}: now reaches U102.26 (IO4)
- net LED_IC: now reaches U102.30 (IO18)
- net ~{I2C_SDA}: now reaches U102.33 (IO21)
- net ~{I2C_SDA}: now also U104.23 (SDA)
- net ~{I2C_SCL}: now reaches U102.36 (IO22)
- net ~{I2C_SCL}: now also U104.22 (SCL)
- net ~{I2C_RESET}: now reaches U102.37 (IO23)
- net ~{I2C_RESET}: now also U104.3 (~{RESET})
- net at R109.1: now also Q101.1 (B); no longer Q101.2 (B)
- net VCC_SWITCH renamed 5V
- new net B_DRAW: SW109.1 (A)
- new net B_END: SW108.1 (A)
- new net B_MOVE: SW107.1 (A)
- new net SCL_DB: OLED102.4 (SDA), R106.2, U104.9 (SC2)
- new net SCL_DM: OLED103.4 (SDA), R111.2, U104.11 (SC3), U104.7 (SC1)
- new net SCL_DW: OLED101.4 (SDA), R105.2
- new net SDA_DB: OLED102.3 (SCL), R108.1, U104.8 (SD2)
- new net SDA_DM: OLED103.3 (SCL), R112.1, U104.10 (SD3), U104.6 (SD1)
- new net SDA_DW: OLED101.3 (SCL), R107.1
- new net SELECT: SW101.1 (A)
- new net SET: SW102.1 (A)
- new net START: SW103.1 (A)
- new net W_DRAW: SW106.1 (A)
- new net W_END: SW105.1 (A)
- new net W_MOVE: SW104.1 (A)
- new net ~{SCL}: U104.5 (SC0)
- new net ~{SDA}: U104.4 (SD0)
- no-connect marks 22 -> 51
Other:
- added sheet Addressable RGB LEDs (rgb_addr_led.kicad_sch)
- added sheet Hall Sensors (hall_sensors.kicad_sch)
- added sheet IO Expander (io_expander_sensor_switches.kicad_sch)
- note added: "Black Chess Clock"
- note added: "I2C Multiplexer"
- note added: "Master Display OLED 128x64"
- note added: "Microprocessor Control Unit ESP32-WROOM-32E (8 MB)"
- note added: "Mounting Holes"
- note added: "Player Clock Display OLED 128x32"
- note added: "Power Switch (DPST)"
- note added: "Shows Game mode, settings, moves, ELO rating, etc."
- note added: "Tactile Buttons"
- note added: "Using I^{2}C multiplexer solve the problem of multiple OLED displays sharing the same device address using the same master I^{2}C bus."
- note added: "White Chess Clock"
- moved on the sheet: J102, U102

Commit message: update schematic with corrections
Parts:
- added C107, C108: (no value), symbol Device:C_Small
- added SW110: (no value), symbol Switch:SW_SPST
Connections:
- net 3V3: now also C107.1, C108.1
- net GND: now also C107.2, C108.2, SW110.2 (B)
- net I2C_A0: now also U102.11 (IO26); no longer U102.10 (IO25)
- net I2C_A1: now also U102.10 (IO25); no longer U102.11 (IO26)
- net SCL_DB: now also U104.11 (SC3); no longer U104.9 (SC2)
- net SCL_DM: no longer U104.11 (SC3)
- net SCL_DW: now also U104.9 (SC2)
- net SDA_DB: now also U104.10 (SD3); no longer U104.8 (SD2)
- net SDA_DM: no longer U104.10 (SD3)
- net SDA_DW: now also U104.8 (SD2)
- net ~{SCL} renamed ~{SCL_IOMUX}
- net ~{SDA} renamed ~{SDA_IOMUX}
- new net MENU: SW110.1 (A)
Other:
- moved on the sheet: SW104, SW105, SW106, SW107, SW108, SW109

Commit message: update schematic to include more components
Added SD card
Added IO expander for tactile buttons
Parts:
- added J103: (no value), symbol Connector:Micro_SD_Card_Det_Hirose_DM3AT
- added J104: (no value), symbol Connector_Generic:Conn_02x03_Odd_Even
- added LED101, LED102, LED103: (no value), symbol Device:LED_Small
- added R113, R114, R115: (no value), symbol Device:R_Small
Connections:
- net 3V3: now also J103.4 (VDD), R113.1, R114.1, R115.1
- net 5V: now also C102.2; no longer C102.1
- net EN: now also J104.1 (Pin_1)
- net GND: now also C102.1, J103.6 (VSS), J104.4 (Pin_4), LED103.1 (K); no longer C102.2
- net IO0: now also J104.6 (Pin_6)
- net VBUS: now also J104.2 (Pin_2)
- net ~{IO_INT}: now also U102.29 (IO5); no longer U102.26 (IO4)
- net SD_SCK: now reaches U102.13 (IO14)
- net SD_SCK: now also J103.5 (CLK)
- net SD_D2: now reaches U102.14 (IO12)
- net SD_D2: now also J103.1 (DAT2)
- net SD_D3: now reaches U102.16 (IO13)
- net SD_D3: now also J103.2 (DAT3/CD)
- net SD_CMD: now reaches U102.23 (IO15)
- net SD_CMD: now also J103.3 (CMD)
- net SD_D0: now reaches U102.24 (IO2)
- net SD_D0: now also J103.7 (DAT0)
- net SD_DET: now reaches U102.27 (IO16)
- net SD_DET: now also J103.9 (DET_B)
- new net: LED101.2 (A), R113.2
- new net: LED102.2 (A), R114.2
- new net: LED103.2 (A), R115.2
- new net RX0: J104.5 (Pin_5), LED101.1 (K)
- new net SD_D1: J103.8 (DAT1), U102.26 (IO4)
- new net TX0: J104.3 (Pin_3), LED102.1 (K)
- no-connect marks 51 -> 46
Other:
- note added: "Backup Programmer"
- note added: "Indicator LEDs"
- note added: "Pin Assignment sck 14 cmd 15 D0 2 D1 4 D2 12 D3 13"
- note added: "SD Card Interface"
- moved on the sheet: C102, C103, C105, C106, H101, H102, H103, H104, H105, H106, H107, H108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

Commit message: change wording from TTL to UART
Other:
- note added: "USB to UART Auto Program Circuit"
- note removed: "USB to TTL Auto Program Circuit"
Changed lines of the file:
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@@
     (effects (font (size 1.5 1.5)) (justify left bottom))
   )
-  (text "USB to TTL\nAuto Program Circuit" (at 107.95 171.45 180)
+  (text "USB to UART\nAuto Program Circuit" (at 107.95 171.45 180)
     (effects (font (size 1.5 1.5) italic) (justify right bottom))
   )

Commit message: update schematics
Parts:
- added R116, R117, R118: (no value), symbol Device:R_Small
- R113, R114: LCSC C17513 -> (none)
- R115: LCSC C17710 -> (none)
Connections:
- net 3V3: now also R116.1, R117.1, R118.1
- net LED_IC: now also U102.28 (IO17); no longer U102.30 (IO18)
- net SD_SCK: now also U102.30 (IO18); no longer U102.13 (IO14)
- net ~{I2C_RESET}: now also U102.26 (IO4); no longer U102.37 (IO23)
- net ~{IO_INT}: now also U102.9 (IO33); no longer U102.29 (IO5)
- net SD_MISO: now reaches U102.31 (IO19)
- net SD_MISO: now also J103.7 (DAT0), R117.2
- net SD_CMD: no longer names the net of U102.23 (IO15)
- net SD_CMD: no longer J103.3 (CMD)
- net SD_D0: no longer names the net of U102.24 (IO2)
- net SD_D0: no longer J103.7 (DAT0)
- net SD_D1: no longer names the net of J103.8 (DAT1)
- net SD_D1: no longer U102.26 (IO4)
- net SD_D2: no longer names the net of U102.14 (IO12)
- net SD_D2: no longer J103.1 (DAT2)
- net SD_D3: no longer names the net of U102.16 (IO13)
- net SD_D3: no longer J103.2 (DAT3/CD)
- new net SD_MOSI: J103.3 (CMD), R118.2, U102.37 (IO23)
- new net SD_SS: J103.2 (DAT3/CD), R116.2, U102.29 (IO5)
- no-connect marks 46 -> 50
Other:
- note added: "Pull-Up Resistors for SD Card SPI BUS"
- note added: "VSPI - SPI Bus D2(SS) 5 CLK 18 D0(MISO) 19 CMD(MOSI) 23"
- note removed: "Pin Assignment sck 14 cmd 15 D0 2 D1 4 D2 12 D3 13"
- moved on the sheet: C107, C108, J103

Commit message: add level translator and fix OLED pin assignment
Parts:
- added R119, R120: (no value), symbol Device:R_Small
- R105, R106, R107, R108, R111, R112: LCSC C23162 -> (none)
Connections:
- net RX0 is gone; now on net RXD: J104.5 (Pin_5), LED101.1 (K)
- net TX0 is gone; now on net TXD: J104.3 (Pin_3), LED102.1 (K)
- net 3V3: now also R105.2, R106.2, R111.2, R119.2, R120.2; no longer R105.1, R106.1, R111.1
- net LED_IC: now also U102.24 (IO2); no longer U102.28 (IO17)
- net SCL_DB: now also OLED102.3 (SCL), R111.1; no longer OLED102.4 (SDA), R106.2
- net SCL_DM: now also OLED103.3 (SCL), R119.1; no longer OLED103.4 (SDA), R111.2
- net SCL_DW: now also OLED101.3 (SCL), R112.1; no longer OLED101.4 (SDA), R105.2
- net SDA_DB: now also OLED102.4 (SDA), R105.1; no longer OLED102.3 (SCL), R108.1
- net SDA_DM: now also OLED103.4 (SDA), R107.1; no longer OLED103.3 (SCL), R112.1
- net SDA_DW: now also OLED101.4 (SDA), R106.1; no longer OLED101.3 (SCL), R107.1
- net ~{SCL_IOMUX}: now also R120.1
- net ~{SDA_IOMUX}: now also R108.1
Other:
- moved on the sheet: OLED101, OLED102, OLED103, U104

Commit message: repurpose design with Nextion display
Parts:
- removed OLED103: (no value), symbol User_Symbols:OLED_I2C
- removed R105, R106, R107, R108, R111, R112, R119, R120: (no value), symbol Device:R_Small
- removed SW101, SW102, SW103, SW110: (no value), symbol Switch:SW_SPST
- added J105: (no value), User Custom Footprint:NX3224T024, symbol User_Symbols:NX3224T024
- C101, C105, C106, C108: value (none) -> 100nF; footprint (none) -> Capacitor_SMD:C_0603_1608Metric
- C102: value (none) -> 22uF; footprint (none) -> Capacitor_SMD:C_0603_1608Metric
- C103: value (none) -> 4.7uF; footprint (none) -> Capacitor_SMD:C_0603_1608Metric
- C104: value (none) -> 4.7nF; footprint (none) -> Capacitor_SMD:C_0603_1608Metric
- C107: value (none) -> 10uF; footprint (none) -> Capacitor_SMD:C_0603_1608Metric
- H101, H102, H103, H104, H105, H106, H107, H108, H109: value (none) -> MountingHole; footprint (none) -> MountingHole:MountingHole_2.7mm_M2.5_ISO7380
- J101: value (none) -> USB_C_Receptacle_USB2.0; footprint (none) -> Connector_USB:USB_C_Receptacle_JAE_DX07S016JA1R1500
- J102: value (none) -> Conn_01x03; footprint (none) -> Connector_PinHeader_2.54mm:PinHeader_1x03_P2.54mm_Vertical
- J103: value (none) -> Micro_SD_Card_Det_Hirose_DM3CS-SF; footprint (none) -> User Custom Footprint:DM3CSSF
- J104: value (none) -> Conn_02x03_Odd_Even; footprint (none) -> Tag_Connect:TC2030-IDC-NL
- LED101: value (none) -> BLUE; footprint (none) -> LED_SMD:LED_0603_1608Metric
- LED102: value (none) -> GREEN; footprint (none) -> LED_SMD:LED_0603_1608Metric
- LED103: value (none) -> RED; footprint (none) -> LED_SMD:LED_0603_1608Metric
- OLED101, OLED102: value (none) -> OLED_I2C; footprint (none) -> User Custom Footprint:OLED_128x32_I2C_4pins
- Q101, Q102: value (none) -> S8050; footprint (none) -> Package_TO_SOT_SMD:SOT-23
- R101, R109, R110, R116, R117, R118: value (none) -> 10K; footprint (none) -> Resistor_SMD:R_0603_1608Metric
- R102, R103: value (none) -> 5K1; footprint (none) -> Resistor_SMD:R_0805_2012Metric
- R104: value (none) -> 1M; footprint (none) -> Resistor_SMD:R_0603_1608Metric
- R113, R114: value (none) -> 1K; footprint (none) -> Resistor_SMD:R_0603_1608Metric
- R115: value (none) -> 470; footprint (none) -> Resistor_SMD:R_0603_1608Metric
- SW104, SW105, SW106, SW107, SW108, SW109: value (none) -> SW_SPST; footprint (none) -> User Custom Footprint:Button_SW_12mm_1.8mm_hole
- U101: value (none) -> XC6220B331MR-G; footprint (none) -> Package_TO_SOT_SMD:SOT-23-5
- U102: value (none) -> ESP32-WROOM-32E; footprint (none) -> RF_Module:ESP32-WROOM-32
- U103: value (none) -> SRV05-4; footprint (none) -> Package_TO_SOT_SMD:SOT-23-6
- U104: value (none) -> PCA9548APW; footprint (none) -> Package_SO:TSSOP-24_4.4x7.8mm_P0.65mm
- U105: value (none) -> CP2102-GMR; footprint (none) -> Package_DFN_QFN:QFN-28-1EP_5x5mm_P0.5mm_EP3.35x3.35mm
Connections:
- net 5V: now also J105.1 (VCC)
- net GND: now also J103.11 (SHIELD), U104.1 (A0), U104.2 (A1), U104.21 (A2), J105.4 (GND)
- net SD_DET: now also U102.13 (IO14); no longer U102.27 (IO16)
- net TX2: now reaches U102.28 (IO17)
- net TX2: now also J105.3 (RX)
- net I2C_A0: no longer names the net of U102.11 (IO26)
- net I2C_A0: no longer U104.1 (A0)
- net I2C_A1: no longer names the net of U102.10 (IO25)
- net I2C_A1: no longer U104.2 (A1)
- net I2C_A2: no longer names the net of U102.12 (IO27)
- net I2C_A2: no longer U104.21 (A2)
- net RXD renamed RX0
- net TXD renamed TX0
- new net RX2: J105.2 (TX), U102.27 (IO16)
Other:
- note added: "By-pass Caps"
- note added: "I2C addr 0x60"
- note added: "I2C addr 0x70"
- note added: "I^{2}C Multiplex Clk"
- note added: "I^{2}C Multiplex Data"
- note added: "I^{2}C Multiplexer"
- note added: "Master Display Nextion 2.4" TFT"
- note added: "Mounting Holes Chess Board Support"
- note added: "Nextion RX"
- note added: "Nextion TX"
- note added: "SD Card"
- note added: "SD Card Detector"
- note added: "SD Card Select"
- note added: "Using I^{2}C multiplexer solve the problem of multiple OLED displays sharing the same device address using the same master I^{2}C bus. Pull-up resistors are not needed since PCA9548APW has built-in voltage translation and is > V_{iH} for target peripherals."
- note removed: "I2C Multiplexer"
- note removed: "Master Display OLED 128x64"
- note removed: "Mounting Holes"
- note removed: "Shows Game mode, settings, moves, ELO rating, etc."
- note removed: "Using I^{2}C multiplexer solve the problem of multiple OLED displays sharing the same device address using the same master I^{2}C bus."
- moved on the sheet: C101, C107, C108, H101, H102, H103, H104, H105, H106, H107, H108, H109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

Commit message: add bypass caps
Parts:
- added C109: (no value), symbol Device:C_Small
- C101, C105, C106, C108: value 100nF -> (none); footprint Capacitor_SMD:C_0603_1608Metric -> (none)
- C102: value 22uF -> (none); footprint Capacitor_SMD:C_0603_1608Metric -> (none)
- C103: value 4.7uF -> (none); footprint Capacitor_SMD:C_0603_1608Metric -> (none)
- C104: value 4.7nF -> (none); footprint Capacitor_SMD:C_0603_1608Metric -> (none)
- C107: value 10uF -> (none); footprint Capacitor_SMD:C_0603_1608Metric -> (none)
- H101, H102, H103, H104, H105, H106, H107, H108, H109: value MountingHole -> (none); footprint MountingHole:MountingHole_2.7mm_M2.5_ISO7380 -> (none)
- J101: value USB_C_Receptacle_USB2.0 -> (none); footprint Connector_USB:USB_C_Receptacle_JAE_DX07S016JA1R1500 -> (none)
- J102: value Conn_01x03 -> (none); footprint Connector_PinHeader_2.54mm:PinHeader_1x03_P2.54mm_Vertical -> (none)
- J103: value Micro_SD_Card_Det_Hirose_DM3CS-SF -> (none); footprint User Custom Footprint:DM3CSSF -> (none)
- J104: value Conn_02x03_Odd_Even -> (none); footprint Tag_Connect:TC2030-IDC-NL -> (none)
- J105: footprint User Custom Footprint:NX3224T024 -> (none); now left out of the parts list
- LED101: value BLUE -> (none); footprint LED_SMD:LED_0603_1608Metric -> (none)
- LED102: value GREEN -> (none); footprint LED_SMD:LED_0603_1608Metric -> (none)
- LED103: value RED -> (none); footprint LED_SMD:LED_0603_1608Metric -> (none)
- OLED101, OLED102: value OLED_I2C -> (none); footprint User Custom Footprint:OLED_128x32_I2C_4pins -> (none); now left out of the parts list
- Q101, Q102: value S8050 -> (none); footprint Package_TO_SOT_SMD:SOT-23 -> (none)
- R101, R109, R110, R116, R117, R118: value 10K -> (none); footprint Resistor_SMD:R_0603_1608Metric -> (none)
- R102, R103: value 5K1 -> (none); footprint Resistor_SMD:R_0805_2012Metric -> (none)
- R104: value 1M -> (none); footprint Resistor_SMD:R_0603_1608Metric -> (none)
- R113, R114: value 1K -> (none); footprint Resistor_SMD:R_0603_1608Metric -> (none)
- R115: value 470 -> (none); footprint Resistor_SMD:R_0603_1608Metric -> (none)
- SW104, SW105, SW106, SW107, SW108, SW109: value SW_SPST -> (none); footprint User Custom Footprint:Button_SW_12mm_1.8mm_hole -> (none)
- U101: value XC6220B331MR-G -> (none); footprint Package_TO_SOT_SMD:SOT-23-5 -> (none)
- U102: value ESP32-WROOM-32E -> (none); footprint RF_Module:ESP32-WROOM-32 -> (none)
- U103: value SRV05-4 -> (none); footprint Package_TO_SOT_SMD:SOT-23-6 -> (none)
- U104: value PCA9548APW -> (none); footprint Package_SO:TSSOP-24_4.4x7.8mm_P0.65mm -> (none)
- U105: value CP2102-GMR -> (none); footprint Package_DFN_QFN:QFN-28-1EP_5x5mm_P0.5mm_EP3.35x3.35mm -> (none)
Connections:
- net 3V3: now also C109.1
- net GND: now also C109.2
