File: chess-board-iot.kicad_sch (KiCad schematic)
At the start: 53 parts

Commit message: refactor power rail
Parts:
- added C111: (no value), symbol Device:C_Small
- added D101: (no value), symbol User_Symbols:RClamp0524PATCT
- added F101: (no value), symbol Device:Polyfuse
- added L101: (no value), symbol Device:L_Ferrite_Small
- added R105: (no value), symbol Device:R_Small
- J102: symbol Connector_Generic:Conn_01x03 -> Switch:SW_SPDT; LCSC (none) -> C319015; now in the parts list
Connections:
- net 3V3: now also R116.2, R117.2, R118.2; no longer R116.1, R117.1, R118.1
- net 5V: now also C105.1, U105.7 (VREGIN), U105.8 (VBUS), C111.1
- net GND: now also C111.2, D101.3 (A)
- net SD_MISO: now also R116.1, D101.1 (K1); no longer R117.2
- net SD_MOSI: now also R117.1, D101.4 (K3); no longer R118.2
- net SD_SCK: now also D101.2 (K2), R105.2; no longer U102.30 (IO18)
- net SD_SS: now also R118.1, D101.5 (K4); no longer R116.2
- net VBUS: now also F101.1; no longer C105.1, J102.2 (Pin_2), U103.5 (VP), U105.7 (VREGIN), U105.8 (VBUS)
- new net: R105.1, U102.30 (IO18)
- new net: F101.2, L101.1
- new net VBUS_Filtered: J102.2 (B), L101.2, U103.5 (VP)
Other:
- note added: "Power Switch (SPDT)"
- note removed: "Power Switch (DPST)"
- note removed: "Power Switch SPDT"
- note removed: "Pull-Up Resistors for SD Card SPI BUS"
- moved on the sheet: C101, C102, C103, C104, C107, C108, H101, H102, H103, H104, H105, H106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

Commit message: fix sd card layout
Parts:
- R105: LCSC (none) -> C107701
- R113, R114: LCSC (none) -> C21190
- R115: LCSC (none) -> C23179
Other:
- moved on the sheet: C101, R101, R105, U102

Commit message: fix USB-C footprint and traces
Parts:
- U102: LCSC C701341 -> C701342
Changed lines of the file:
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@@
       (effects (font (size 1.27 1.27)) hide)
     )
-    (property "LCSC" "C701341" (id 4) (at 285.75 57.15 0)
+    (property "LCSC" "C701342" (id 4) (at 285.75 57.15 0)
       (effects (font (size 1.27 1.27)) hide)
     )
@@
     )
     (path "/582a69f8-5434-4554-917e-70d2bc28584c"
-      (reference "J101") (unit 1) (value "USB_C_Receptacle_USB2.0") (footprint "Connector_USB:USB_C_Receptacle_JAE_DX07S016JA1R1500")
+      (reference "J101") (unit 1) (value "USB_C_Receptacle_USB2.0") (footprint "User Custom Footprint:USB_C_Receptable_918-418K2023S40001")
     )
     (path "/64f954f3-8828-4c30-b54d-fa7a7ce114c2"
@@
     )
     (path "/7531744a-adfd-462a-a28f-135299bc08b0"
-      (reference "U102") (unit 1) (value "ESP32-WROOM-32E") (footprint "RF_Module:ESP32-WROOM-32")
+      (reference "U102") (unit 1) (value "ESP32-WROOM-32E (8MB)") (footprint "RF_Module:ESP32-WROOM-32")
     )
     (path "/bbc54aa5-5efc-46ea-83fa-f9acfbcc058f"

Commit message: add buck converter, switch ESD component
Parts:
- removed J102: (no value), symbol Switch:SW_SPDT
- added R106, R107, R108, R111, R112: (no value), symbol Device:R_Small
- C104: LCSC C53987 -> C14663
- C107: LCSC C15850 -> C59461
- R104: LCSC C22935 -> C13167
- U103: symbol Power_Protection:SRV05-4 -> Power_Protection:SP0503BAHT; LCSC C85364 -> C151299
Connections:
- net 3V3: now also R104.1, R106.1, R107.1, R108.1, R111.1, R112.1; no longer C106.1, U105.6 (VDD)
- net 5V: now also C104.1, L101.2
- net D_P: now also U103.2 (K); no longer U103.1 (IO1)
- net GND: now also U103.1 (A); no longer R104.1, U103.2 (VN)
- net SCL_DB: now also R111.2
- net SCL_DW: now also R107.2
- net SDA_DB: now also R112.2
- net SDA_DW: now also R108.2
- net VBUS: now also U103.4 (K)
- net ~{SCL_IOMUX}: now also R104.2
- net ~{SDA_IOMUX}: now also R106.2
- net SCL_DM: no longer names the net of U104.7 (SC1)
- net SDA_DM: no longer names the net of U104.6 (SD1)
- removed net VBUS_Filtered: L101.2, U103.5 (VP)
- new net: C106.1, U105.6 (VDD)
- now unconnected: J101.S1 (SHIELD)
Other:
- added sheet Buck Converter (buck_converter.kicad_sch)
- note added: "Backup Programmer ESP-PROG"
- note added: "By-pass Caps Pin 2"
- note added: "By-pass Caps Pin 24"
- note added: "By-pass Caps Pin 7,8"
- note removed: "Backup Programmer"
- note removed: "By-pass Caps"
- note removed: "Off"
- note removed: "On"
- note removed: "Power Switch (SPDT)"
- moved on the sheet: C105, C106, C109, F101, J101, J104, L101, R102, R103, U104, U105

Commit message: remove buck converter schematic
Moved to separate branch
Other:
- removed sheet Buck Converter
Changed lines of the file:
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@@
   (title_block
     (title "Chess Board IOT")
-    (date "2022-10-13")
+    (date "2022-10-17")
     (rev "A")
     (company "Butler Electronics")
@@
     (pin "1")
   )
-  (sheet (at 124.46 177.8) (size 33.02 22.86) (fields_autoplaced)
-    (stroke (width 0.1524) (type solid) (color 0 0 0 0))
-    (fill (color 0 0 0 0.0000))
-    (property "Sheet name" "Buck Converter" (id 0) (at 124.46 177.0884 0)
-      (effects (font (size 1.27 1.27)) (justify left bottom))
-    )
-    (property "Sheet file" "buck_converter.kicad_sch" (id 1) (at 124.46 201.2446 0)
-      (effects (font (size 1.27 1.27)) (justify left top) hide)
-    )
-  )
   (sheet (at 13.97 177.8) (size 33.02 22.86) (fields_autoplaced)
     (stroke (width 0.1524) (type solid) (color 0 0 0 0))
@@
     (path "/dd7b36d6-edb3-405d-85c2-82cc4203666c" (page "4"))
     (path "/bee0bfe3-a22e-4053-aac2-d61040bc25d4" (page "5"))
-    (path "/2cba3c02-6621-4821-9c99-ae1947b33125" (page "5"))
   )
   (symbol_instances
@@
       (reference "#PWR0108") (unit 1) (value "GND") (footprint "")
     )
-    (path "/2cba3c02-6621-4821-9c99-ae1947b33125/4054bf7c-ed95-422f-9780-32ad24300a9e"
-      (reference "#PWR0109") (unit 1) (value "GND") (footprint "")
-    )
-    (path "/2cba3c02-6621-4821-9c99-ae1947b33125/3ca443f0-ea30-4925-8d82-08f3e9f10fcb"
-      (reference "#PWR0110") (unit 1) (value "GND") (footprint "")
-    )
     (path "/5dbfae8c-9480-475b-9278-829262d21cce"
       (reference "#PWR0111") (unit 1) (value "GND") (footprint "")
@@
       (reference "C464") (unit 1) (value "100nF") (footprint "Capacitor_SMD:C_0603_1608Metric")
     )
-    (path "/2cba3c02-6621-4821-9c99-ae1947b33125/c556e849-514e-4d94-baaa-e2fb49152ab8"
-      (reference "C501") (unit 1) (value "100nF") (footprint "Capacitor_SMD:C_0603_1608Metric")
-    )
-    (path "/2cba3c02-6621-4821-9c99-ae1947b33125/3baea911-fc9a-4a51-856e-07dd7478443a"
-      (reference "C502") (unit 1) (value "10uF") (footprint "Capacitor_SMD:C_0603_1608Metric")
-    )
-    (path "/2cba3c02-6621-4821-9c99-ae1947b33125/07cc2cf1-d7f1-4c11-8fc2-85d63de65da1"
-      (reference "C503") (unit 1) (value "100uF") (footprint "Capacitor_SMD:C_0603_1608Metric")
-    )
-    (path "/2cba3c02-6621-4821-9c99-ae1947b33125/83314601-2f7d-4108-8e80-462f4afb2566"
-      (reference "C504") (unit 1) (value "100uF") (footprint "Capacitor_SMD:C_0603_1608Metric")
-    )
-    (path "/2cba3c02-6621-4821-9c99-ae1947b33125/f8f0f618-0ffd-4dc3-bae2-7c0a6807c2e1"
-      (reference "C505") (unit 1) (value "10pF") (footprint "Capacitor_SMD:C_0603_1608Metric")
-    )
-    (path "/2cba3c02-6621-4821-9c99-ae1947b33125/25ac1e61-34ec-4246-b7f9-bfecc2bb509d"
-      (reference "C506") (unit 1) (value "1nF") (footprint "Capacitor_SMD:C_0603_1608Metric")
-    )
-    (path "/2cba3c02-6621-4821-9c99-ae1947b33125/2ef7a46f-1777-4e41-84ce-5811a5faa597"
-      (reference "C507") (unit 1) (value "8.2nF") (footprint "Capacitor_SMD:C_0603_1608Metric")
-    )
     (path "/49a9d7f1-a588-4ad2-b5d1-ad10c25e1b2b"
       (reference "D101") (unit 1) (value "RClamp0524PATCT") (footprint "User Custom Footprint:SLP2510P8")
@@
       (reference "D264") (unit 1) (value "WS2813C") (footprint "LED_SMD:LED_WS2812_PLCC6_5.0x5.0mm_P1.6mm")
     )
-    (path "/2cba3c02-6621-4821-9c99-ae1947b33125/87e412d9-78da-45ea-bf20-817fea246726"
-      (reference "D501") (unit 1) (value "D_Schottky_Small") (footprint "Diode_SMD:D_SMA")
-    )
     (path "/93db65ef-2998-46f8-9a92-6ea4cd0e8ae5"
       (reference "F101") (unit 1) (value "C207047") (footprint "Fuse:Fuse_1210_3225Metric")
@@
       (reference "L101") (unit 1) (value "L_Ferrite_Small") (footprint "Inductor_SMD:L_0805_2012Metric_Pad1.15x1.40mm_HandSolder")
     )
-    (path "/2cba3c02-6621-4821-9c99-ae1947b33125/2824ab54-428a-4677-baff-74b7123166dc"
-      (reference "L501") (unit 1) (value "3.3uH") (footprint "User Custom Footprint:L_4.0x4.0_H2.6")
-    )
     (path "/1f67b0ac-5c7d-4dd9-80c1-04c16b0192e4"
       (reference "LED101") (unit 1) (value "BLUE") (footprint "LED_SMD:LED_0603_1608Metric")
@@
       (reference "R464") (unit 1) (value "2K7") (footprint "Resistor_SMD:R_0603_1608Metric")
     )
-    (path "/2cba3c02-6621-4821-9c99-ae1947b33125/5bca96fa-d004-4c9a-80c2-af95bf154d29"
-      (reference "R501") (unit 1) (value "10K2") (footprint "Resistor_SMD:R_0603_1608Metric")
-    )
-    (path "/2cba3c02-6621-4821-9c99-ae1947b33125/1cc83fe6-5359-419f-9a58-a72b62e54cf6"
-      (reference "R502") (unit 1) (value "24K9") (footprint "Resistor_SMD:R_0603_1608Metric")
-    )
-    (path "/2cba3c02-6621-4821-9c99-ae1947b33125/fd3d4681-fe68-462e-8583-9b8d3cb1987e"
-      (reference "R503") (unit 1) (value "3K24") (footprint "Resistor_SMD:R_0603_1608Metric")
-    )
     (path "/3eee5851-fa4c-4797-81b3-a82a514a8268"
       (reference "SW104") (unit 1) (value "SW_SPST") (footprint "User Custom Footprint:Button_SW_12mm_1.8mm_hole")
@@
       (reference "U464") (unit 1) (value "UHE4913") (footprint "User Custom Footprint:SOT-23-12_Flipped")
     )
-    (path "/2cba3c02-6621-4821-9c99-ae1947b33125/cac9c82e-7499-4f7f-b4fc-0f389d140e7f"
-      (reference "U501") (unit 1) (value "TPS54331DR") (footprint "Package_SO:SOIC-8_3.9x4.9mm_P1.27mm")
-    )
   )

Commit message: add pull ups, bypass caps for SD card
Parts:
- added C110, C112: (no value), symbol Device:C_Small
- added H110, H111, H112, H113, H114, H115: (no value), symbol Mechanical:MountingHole
- added R119, R120: (no value), symbol Device:R_Small
- R116, R117, R118: LCSC C25804 -> C25819
Connections:
- net 3V3: now also C110.1, C112.1, R119.2, R120.2
- net GND: now also C110.2, C112.2
- net SD_MISO: now also R105.1; no longer J103.7 (DAT0)
- net SD_SCK: now also U102.30 (IO18); no longer R105.2
- net at J103.1 (DAT2): now also R120.1
- net at J103.8 (DAT1): now also R119.1
- new net: J103.7 (DAT0), R105.2
- no-connect marks 50 -> 48
Other:
- note added: "By-pass Caps Pin 4"
- note added: "Chessboard"
- note added: "PCB Board"
- moved on the sheet: C102, C103, D101, H101, H102, H103, H104, H105, H106, H107, H108, H109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

Commit message: add pull ups, bypass caps for SD card
Parts:
- removed R105: (no value), symbol Device:R_Small
- C101, C105, C106, C108, C109, C111, C112: value (none) -> 100nF; footprint (none) -> Capacitor_SMD:C_0603_1608Metric
- C102, C107: value (none) -> 22uF; footprint (none) -> Capacitor_SMD:C_0603_1608Metric
- C103: value (none) -> 4.7uF; footprint (none) -> Capacitor_SMD:C_0603_1608Metric
- C104: value (none) -> 1uF; footprint (none) -> Capacitor_SMD:C_0603_1608Metric
- C110: value (none) -> 10uF; footprint (none) -> Capacitor_SMD:C_0603_1608Metric
- D101: value (none) -> RClamp0524PATCT; footprint (none) -> User Custom Footprint:SLP2510P8
- F101: value (none) -> C207047; footprint (none) -> Fuse:Fuse_1210_3225Metric
- H101, H102, H103, H104, H105, H106, H107, H108, H109: value (none) -> MountingHole; footprint (none) -> MountingHole:MountingHole_2.7mm_M2.5_ISO7380
- H110, H111, H112, H113, H114, H115: value (none) -> MountingHole; footprint (none) -> MountingHole:MountingHole_3.2mm_M3_ISO7380_Pad
- J101: value (none) -> USB_C_Receptacle_USB2.0; footprint (none) -> User Custom Footprint:USB_C_Receptable_918-418K2023S40001
- J103: value (none) -> Micro_SD_Card_Det_Hirose_DM3CS-SF; footprint (none) -> User Custom Footprint:DM3CS-SF
- J104: value (none) -> Conn_02x03_Odd_Even; footprint (none) -> Tag_Connect:TC2030-IDC-NL
- J105: value (none) -> NX3224T024; footprint (none) -> User Custom Footprint:NX3224T024
- L101: value (none) -> L_Ferrite_Small; footprint (none) -> Inductor_SMD:L_0805_2012Metric_Pad1.15x1.40mm_HandSolder
- LED101: value (none) -> BLUE; footprint (none) -> LED_SMD:LED_0603_1608Metric
- LED102: value (none) -> GREEN; footprint (none) -> LED_SMD:LED_0603_1608Metric
- LED103: value (none) -> RED; footprint (none) -> LED_SMD:LED_0603_1608Metric
- OLED101, OLED102: value (none) -> OLED_I2C; footprint (none) -> User Custom Footprint:OLED_128x32_I2C_4pins
- Q101, Q102: value (none) -> S8050; footprint (none) -> Package_TO_SOT_SMD:SOT-23
- R101, R109, R110: value (none) -> 10K; footprint (none) -> Resistor_SMD:R_0603_1608Metric
- R102, R103: value (none) -> 5K1; footprint (none) -> Resistor_SMD:R_0805_2012Metric
- R104, R106, R107, R108, R111, R112: value (none) -> 2K7; footprint (none) -> Resistor_SMD:R_0603_1608Metric
- R113, R114: value (none) -> 1K; footprint (none) -> Resistor_SMD:R_0603_1608Metric
- R115: value (none) -> 470; footprint (none) -> Resistor_SMD:R_0603_1608Metric
- R116, R117, R118, R119, R120: value (none) -> 47K; footprint (none) -> Resistor_SMD:R_0603_1608Metric
- SW104, SW105, SW106, SW107, SW108, SW109: value (none) -> SW_SPST; footprint (none) -> User Custom Footprint:Button_SW_12mm_1.8mm_hole
- U101: value (none) -> XC6220B331MR-G; footprint (none) -> Package_TO_SOT_SMD:SOT-23-5
- U102: value (none) -> ESP32-WROOM-32E (8MB); footprint (none) -> RF_Module:ESP32-WROOM-32
- U103: value (none) -> SP0503BAHT; footprint (none) -> Package_TO_SOT_SMD:SOT-143
- U104: value (none) -> PCA9548APW; footprint (none) -> Package_SO:TSSOP-24_4.4x7.8mm_P0.65mm
- U105: value (none) -> CP2102-GMR; footprint (none) -> Package_DFN_QFN:QFN-28-1EP_5x5mm_P0.5mm_EP3.35x3.35mm
Connections:
- net SD_MISO: now also J103.7 (DAT0)
