File: chess-board-iot.kicad_sch (KiCad schematic)
At the start: 71 parts, among them J101 USB_C_Receptacle_USB2.0, J103 Micro_SD_Card_Det_Hirose_DM3C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, J104 Conn_02x03_Odd_Even, J105 NX3224T024, Q101 S8050, Q102 S8050, SW104 SW_SPST, SW105 SW_SPST, SW106 SW_SPST, SW107 SW_SPST, SW108 SW_SPST, SW109 SW_SPST, U101 XC6220B331MR-G, U102 ESP32-WROOM-32E (8MB), U103 SP0503BAHT, U104 PCA9548APW, U105 CP2102-GMR

Commit message: update improved layout
Parts:
- H110, H111, H112, H113, H114, H115: value MountingHole -> (none); footprint MountingHole:MountingHole_3.2mm_M3_ISO7380_Pad -> (none); now left out of the parts list
Changed lines of the file:
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@@
   )
   (symbol (lib_id "Mechanical:MountingHole") (at 129.54 157.48 0) (unit 1)
-    (in_bom yes) (on_board yes) (fields_autoplaced)
+    (in_bom no) (on_board yes) (fields_autoplaced)
     (property "Reference" "H111" (id 0) (at 132.08 157.4799 0)
       (effects (font (size 1.27 1.27)) (justify left))
     )
-    (property "Value" "MountingHole" (id 1) (at 132.08 158.7499 0)
+    (property "Value" "" (id 1) (at 132.08 158.7499 0)
       (effects (font (size 1.27 1.27)) (justify left) hide)
     )
-    (property "Footprint" "MountingHole:MountingHole_3.2mm_M3_ISO7380_Pad" (id 2) (at 129.54 157.48 0)
+    (property "Footprint" "" (id 2) (at 129.54 157.48 0)
       (effects (font (size 1.27 1.27)) hide)
     )
@@
   )
   (symbol (lib_id "Mechanical:MountingHole") (at 115.57 157.48 0) (unit 1)
-    (in_bom yes) (on_board yes) (fields_autoplaced)
+    (in_bom no) (on_board yes) (fields_autoplaced)
     (property "Reference" "H110" (id 0) (at 118.11 157.4799 0)
       (effects (font (size 1.27 1.27)) (justify left))
     )
-    (property "Value" "MountingHole" (id 1) (at 118.11 158.7499 0)
+    (property "Value" "" (id 1) (at 118.11 158.7499 0)
       (effects (font (size 1.27 1.27)) (justify left) hide)
     )
-    (property "Footprint" "MountingHole:MountingHole_3.2mm_M3_ISO7380_Pad" (id 2) (at 115.57 157.48 0)
+    (property "Footprint" "" (id 2) (at 115.57 157.48 0)
       (effects (font (size 1.27 1.27)) hide)
     )
@@
   )
   (symbol (lib_id "Mechanical:MountingHole") (at 115.57 162.56 0) (unit 1)
-    (in_bom yes) (on_board yes) (fields_autoplaced)
+    (in_bom no) (on_board yes) (fields_autoplaced)
     (property "Reference" "H113" (id 0) (at 118.11 162.5599 0)
       (effects (font (size 1.27 1.27)) (justify left))
     )
-    (property "Value" "MountingHole" (id 1) (at 118.11 163.8299 0)
+    (property "Value" "" (id 1) (at 118.11 163.8299 0)
       (effects (font (size 1.27 1.27)) (justify left) hide)
     )
-    (property "Footprint" "MountingHole:MountingHole_3.2mm_M3_ISO7380_Pad" (id 2) (at 115.57 162.56 0)
+    (property "Footprint" "" (id 2) (at 115.57 162.56 0)
       (effects (font (size 1.27 1.27)) hide)
     )
@@
   )
   (symbol (lib_id "Mechanical:MountingHole") (at 143.51 157.48 0) (unit 1)
-    (in_bom yes) (on_board yes) (fields_autoplaced)
+    (in_bom no) (on_board yes) (fields_autoplaced)
     (property "Reference" "H112" (id 0) (at 146.05 157.4799 0)
       (effects (font (size 1.27 1.27)) (justify left))
     )
-    (property "Value" "MountingHole" (id 1) (at 146.05 158.7499 0)
+    (property "Value" "" (id 1) (at 146.05 158.7499 0)
       (effects (font (size 1.27 1.27)) (justify left) hide)
     )
-    (property "Footprint" "MountingHole:MountingHole_3.2mm_M3_ISO7380_Pad" (id 2) (at 143.51 157.48 0)
+    (property "Footprint" "" (id 2) (at 143.51 157.48 0)
       (effects (font (size 1.27 1.27)) hide)
     )
@@
   )
   (symbol (lib_id "Mechanical:MountingHole") (at 129.54 162.56 0) (unit 1)
-    (in_bom yes) (on_board yes) (fields_autoplaced)
+    (in_bom no) (on_board yes) (fields_autoplaced)
     (property "Reference" "H114" (id 0) (at 132.08 162.5599 0)
       (effects (font (size 1.27 1.27)) (justify left))
     )
-    (property "Value" "MountingHole" (id 1) (at 132.08 163.8299 0)
+    (property "Value" "" (id 1) (at 132.08 163.8299 0)
       (effects (font (size 1.27 1.27)) (justify left) hide)
     )
-    (property "Footprint" "MountingHole:MountingHole_3.2mm_M3_ISO7380_Pad" (id 2) (at 129.54 162.56 0)
+    (property "Footprint" "" (id 2) (at 129.54 162.56 0)
       (effects (font (size 1.27 1.27)) hide)
     )
@@
   )
   (symbol (lib_id "Mechanical:MountingHole") (at 143.51 162.56 0) (unit 1)
-    (in_bom yes) (on_board yes) (fields_autoplaced)
+    (in_bom no) (on_board yes) (fields_autoplaced)
     (property "Reference" "H115" (id 0) (at 146.05 162.5599 0)
       (effects (font (size 1.27 1.27)) (justify left))
     )
-    (property "Value" "MountingHole" (id 1) (at 146.05 163.8299 0)
+    (property "Value" "" (id 1) (at 146.05 163.8299 0)
       (effects (font (size 1.27 1.27)) (justify left) hide)
     )
-    (property "Footprint" "MountingHole:MountingHole_3.2mm_M3_ISO7380_Pad" (id 2) (at 143.51 162.56 0)
-      (effects (font (size 1.27 1.27)) hide)
-    )
+    (property "Footprint" "" (id 2) (at 143.51 162.56 0)
+      (effects (font (size 1.27 1.27)) hide)
+    )

Commit message: update part
Parts:
- H110, H111, H112, H113, H114, H115: value (none) -> MountingHole; footprint (none) -> MountingHole:MountingHole_3.2mm_M3_ISO7380_Pad
- U103: LCSC C151299 -> C3029025
Changed lines of the file:
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@@
   )
   (text "Microprocessor Control Unit\nESP32-WROOM-32E (8 MB)"
-    (at 340.36 96.52 0)
+    (at 340.36 96.52 180)
     (effects (font (size 1.5 1.5) italic) (justify right bottom))
   )
@@
       (effects (font (size 1.27 1.27)) (justify left))
     )
-    (property "Value" "" (id 1) (at 132.08 158.7499 0)
-      (effects (font (size 1.27 1.27)) (justify left) hide)
-    )
-    (property "Footprint" "" (id 2) (at 129.54 157.48 0)
+    (property "Value" "MountingHole" (id 1) (at 132.08 158.7499 0)
+      (effects (font (size 1.27 1.27)) (justify left) hide)
+    )
+    (property "Footprint" "MountingHole:MountingHole_3.2mm_M3_ISO7380_Pad" (id 2) (at 129.54 157.48 0)
       (effects (font (size 1.27 1.27)) hide)
     )
@@
       (effects (font (size 1.27 1.27)) (justify left))
     )
-    (property "Value" "" (id 1) (at 118.11 158.7499 0)
-      (effects (font (size 1.27 1.27)) (justify left) hide)
-    )
-    (property "Footprint" "" (id 2) (at 115.57 157.48 0)
+    (property "Value" "MountingHole" (id 1) (at 118.11 158.7499 0)
+      (effects (font (size 1.27 1.27)) (justify left) hide)
+    )
+    (property "Footprint" "MountingHole:MountingHole_3.2mm_M3_ISO7380_Pad" (id 2) (at 115.57 157.48 0)
       (effects (font (size 1.27 1.27)) hide)
     )
@@
       (effects (font (size 1.27 1.27)) (justify left))
     )
-    (property "Value" "" (id 1) (at 118.11 163.8299 0)
-      (effects (font (size 1.27 1.27)) (justify left) hide)
-    )
-    (property "Footprint" "" (id 2) (at 115.57 162.56 0)
+    (property "Value" "MountingHole" (id 1) (at 118.11 163.8299 0)
+      (effects (font (size 1.27 1.27)) (justify left) hide)
+    )
+    (property "Footprint" "MountingHole:MountingHole_3.2mm_M3_ISO7380_Pad" (id 2) (at 115.57 162.56 0)
       (effects (font (size 1.27 1.27)) hide)
     )
@@
       (effects (font (size 1.27 1.27)) hide)
     )
-    (property "LCSC" "C151299" (id 4) (at 62.23 63.5 0)
+    (property "LCSC" "C3029025" (id 4) (at 62.23 63.5 0)
       (effects (font (size 1.27 1.27)) hide)
     )
@@
       (effects (font (size 1.27 1.27)) (justify left))
     )
-    (property "Value" "" (id 1) (at 146.05 158.7499 0)
-      (effects (font (size 1.27 1.27)) (justify left) hide)
-    )
-    (property "Footprint" "" (id 2) (at 143.51 157.48 0)
+    (property "Value" "MountingHole" (id 1) (at 146.05 158.7499 0)
+      (effects (font (size 1.27 1.27)) (justify left) hide)
+    )
+    (property "Footprint" "MountingHole:MountingHole_3.2mm_M3_ISO7380_Pad" (id 2) (at 143.51 157.48 0)
       (effects (font (size 1.27 1.27)) hide)
     )
@@
       (effects (font (size 1.27 1.27)) (justify left))
     )
-    (property "Value" "" (id 1) (at 132.08 163.8299 0)
-      (effects (font (size 1.27 1.27)) (justify left) hide)
-    )
-    (property "Footprint" "" (id 2) (at 129.54 162.56 0)
+    (property "Value" "MountingHole" (id 1) (at 132.08 163.8299 0)
+      (effects (font (size 1.27 1.27)) (justify left) hide)
+    )
+    (property "Footprint" "MountingHole:MountingHole_3.2mm_M3_ISO7380_Pad" (id 2) (at 129.54 162.56 0)
       (effects (font (size 1.27 1.27)) hide)
     )
@@
       (effects (font (size 1.27 1.27)) (justify left))
     )
-    (property "Value" "" (id 1) (at 146.05 163.8299 0)
-      (effects (font (size 1.27 1.27)) (justify left) hide)
-    )
-    (property "Footprint" "" (id 2) (at 143.51 162.56 0)
-      (effects (font (size 1.27 1.27)) hide)
-    )
+    (property "Value" "MountingHole" (id 1) (at 146.05 163.8299 0)
+      (effects (font (size 1.27 1.27)) (justify left) hide)
+    )
+    (property "Footprint" "MountingHole:MountingHole_3.2mm_M3_ISO7380_Pad" (id 2) (at 143.51 162.56 0)
+      (effects (font (size 1.27 1.27)) hide)
+    )

Commit message: update footprint
Parts:
- U103: footprint Package_TO_SOT_SMD:SOT-143 -> User Custom Footprint:SOT-143-4
Changed lines of the file:
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@@
       (effects (font (size 1.27 1.27)) (justify left))
     )
-    (property "Footprint" "Package_TO_SOT_SMD:SOT-143" (id 2) (at 67.945 64.77 0)
+    (property "Footprint" "User Custom Footprint:SOT-143-4" (id 2) (at 67.945 64.77 0)
       (effects (font (size 1.27 1.27)) (justify left) hide)
     )
@@
     )
     (path "/bbc54aa5-5efc-46ea-83fa-f9acfbcc058f"
-      (reference "U103") (unit 1) (value "SP0503BAHT") (footprint "Package_TO_SOT_SMD:SOT-143")
+      (reference "U103") (unit 1) (value "SP0503BAHT") (footprint "User Custom Footprint:SOT-143-4")
     )
     (path "/a8872555-0f46-431c-a343-cfc377bc0ae4"

Commit message: update part number for ESD
Parts:
- U103: LCSC C3029025 -> C7074
Changed lines of the file:
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@@
       (effects (font (size 1.27 1.27)) hide)
     )
-    (property "LCSC" "C3029025" (id 4) (at 62.23 63.5 0)
+    (property "LCSC" "C7074" (id 4) (at 62.23 63.5 0)
       (effects (font (size 1.27 1.27)) hide)
     )

Commit message: flip TX/RX pins for programmer port
Connections:
- net RX0: now also J104.3 (Pin_3); no longer J104.5 (Pin_5)
- net TX0: now also J104.5 (Pin_5); no longer J104.3 (Pin_3)
Changed lines of the file:
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@@
     (effects (font (size 1.27 1.27)) (justify right bottom))
   )
-  (label "TX0" (at 118.11 74.93 0)
+  (label "TX0" (at 118.11 77.47 0)
     (effects (font (size 1.27 1.27)) (justify left bottom))
   )
@@
     (effects (font (size 1.27 1.27)) (justify right bottom))
   )
-  (label "RX0" (at 118.11 77.47 0)
+  (label "RX0" (at 118.11 74.93 0)
     (effects (font (size 1.27 1.27)) (justify left bottom))
   )
