File: io_expander_sensor_switches.kicad_sch (KiCad schematic)
At the start: 8 parts

Commit message: update schematic with corrections
Connections:
- net ~{SCL} renamed ~{SCL_IOMUX}
- net ~{SDA} renamed ~{SDA_IOMUX}
Changed lines of the file:
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@@
     (stroke (width 0) (type default) (color 0 0 0 0))
   )
-  (global_label "~{SCL}" (shape input) (at 157.48 113.03 180) (fields_autoplaced)
+  (global_label "~{SCL_IOMUX}" (shape input) (at 157.48 113.03 180) (fields_autoplaced)
     (effects (font (size 1.27 1.27)) (justify right))
     (property "Intersheet References" "${INTERSHEET_REFS}" (id 0) (at 151.5593 112.9506 0)
@@
     )
   )
-  (global_label "~{SDA}" (shape bidirectional) (at 157.48 34.29 180) (fields_autoplaced)
+  (global_label "~{SDA_IOMUX}" (shape bidirectional) (at 157.48 34.29 180) (fields_autoplaced)
     (effects (font (size 1.27 1.27)) (justify right))
     (property "Intersheet References" "${INTERSHEET_REFS}" (id 0) (at 151.4988 34.2106 0)
@@
     )
   )
-  (global_label "~{SCL}" (shape input) (at 157.48 36.83 180) (fields_autoplaced)
+  (global_label "~{SCL_IOMUX}" (shape input) (at 157.48 36.83 180) (fields_autoplaced)
     (effects (font (size 1.27 1.27)) (justify right))
     (property "Intersheet References" "${INTERSHEET_REFS}" (id 0) (at 151.5593 36.7506 0)
@@
     )
   )
-  (global_label "~{SDA}" (shape bidirectional) (at 76.2 34.29 180) (fields_autoplaced)
+  (global_label "~{SDA_IOMUX}" (shape bidirectional) (at 76.2 34.29 180) (fields_autoplaced)
     (effects (font (size 1.27 1.27)) (justify right))
     (property "Intersheet References" "${INTERSHEET_REFS}" (id 0) (at 70.2188 34.2106 0)
@@
     )
   )
-  (global_label "~{SDA}" (shape bidirectional) (at 157.48 110.49 180) (fields_autoplaced)
+  (global_label "~{SDA_IOMUX}" (shape bidirectional) (at 157.48 110.49 180) (fields_autoplaced)
     (effects (font (size 1.27 1.27)) (justify right))
     (property "Intersheet References" "${INTERSHEET_REFS}" (id 0) (at 151.4988 110.4106 0)
@@
     )
   )
-  (global_label "~{SCL}" (shape input) (at 76.2 36.83 180) (fields_autoplaced)
+  (global_label "~{SCL_IOMUX}" (shape input) (at 76.2 36.83 180) (fields_autoplaced)
     (effects (font (size 1.27 1.27)) (justify right))
     (property "Intersheet References" "${INTERSHEET_REFS}" (id 0) (at 70.2793 36.7506 0)
@@
     )
   )
-  (global_label "~{SCL}" (shape input) (at 76.2 113.03 180) (fields_autoplaced)
+  (global_label "~{SCL_IOMUX}" (shape input) (at 76.2 113.03 180) (fields_autoplaced)
     (effects (font (size 1.27 1.27)) (justify right))
     (property "Intersheet References" "${INTERSHEET_REFS}" (id 0) (at 70.2793 112.9506 0)
@@
     )
   )
-  (global_label "~{SDA}" (shape bidirectional) (at 76.2 110.49 180) (fields_autoplaced)
+  (global_label "~{SDA_IOMUX}" (shape bidirectional) (at 76.2 110.49 180) (fields_autoplaced)
     (effects (font (size 1.27 1.27)) (justify right))
     (property "Intersheet References" "${INTERSHEET_REFS}" (id 0) (at 70.2188 110.4106 0)
@@
       (effects (font (size 1.27 1.27)) hide)
     )
-    (property "Value" "" (id 1) (at 97.79 163.83 0)
+    (property "Value" "GND" (id 1) (at 97.79 163.83 0)
       (effects (font (size 1.27 1.27)) hide)
     )
@@
       (effects (font (size 1.27 1.27)) hide)
     )
-    (property "Value" "" (id 1) (at 76.2 87.63 0)
+    (property "Value" "GND" (id 1) (at 76.2 87.63 0)
       (effects (font (size 1.27 1.27)) hide)
     )
@@
       (effects (font (size 1.27 1.27)) hide)
     )
-    (property "Value" "" (id 1) (at 76.2 163.83 0)
+    (property "Value" "GND" (id 1) (at 76.2 163.83 0)
       (effects (font (size 1.27 1.27)) hide)
     )
@@
       (effects (font (size 1.27 1.27)) hide)
     )
-    (property "Value" "" (id 1) (at 97.79 87.63 0)
+    (property "Value" "GND" (id 1) (at 97.79 87.63 0)
       (effects (font (size 1.27 1.27)) hide)
     )
@@
       (effects (font (size 1.27 1.27)) hide)
     )
-    (property "Value" "" (id 1) (at 157.48 87.63 0)
+    (property "Value" "GND" (id 1) (at 157.48 87.63 0)
       (effects (font (size 1.27 1.27)) hide)
     )
@@
       (effects (font (size 1.27 1.27)) hide)
     )
-    (property "Value" "" (id 1) (at 179.07 163.83 0)
+    (property "Value" "GND" (id 1) (at 179.07 163.83 0)
       (effects (font (size 1.27 1.27)) hide)
     )
@@
       (effects (font (size 1.27 1.27)) hide)
     )
-    (property "Value" "" (id 1) (at 179.07 87.63 0)
+    (property "Value" "GND" (id 1) (at 179.07 87.63 0)
       (effects (font (size 1.27 1.27)) hide)
     )
@@
       (effects (font (size 1.27 1.27)) hide)
     )
-    (property "Value" "" (id 1) (at 157.48 163.83 0)
-      (effects (font (size 1.27 1.27)) hide)
-    )
+    (property "Value" "GND" (id 1) (at 157.48 163.83 0)
+      (effects (font (size 1.27 1.27)) hide)
+    )

Commit message: refactor IO expander pin assignment
Connections:
- net Tile_09: now also U301.17 (P14); no longer U301.13 (P10)
- net Tile_10: now also U301.18 (P15); no longer U301.14 (P11)
- net Tile_11: now also U301.19 (P16); no longer U301.15 (P12)
- net Tile_12: now also U301.20 (P17); no longer U301.16 (P13)
- net Tile_13: now also U301.13 (P10); no longer U301.17 (P14)
- net Tile_14: now also U301.14 (P11); no longer U301.18 (P15)
- net Tile_15: now also U301.15 (P12); no longer U301.19 (P16)
- net Tile_16: now also U301.16 (P13); no longer U301.20 (P17)
- net Tile_25: now also U302.17 (P14); no longer U302.13 (P10)
- net Tile_26: now also U302.18 (P15); no longer U302.14 (P11)
- net Tile_27: now also U302.19 (P16); no longer U302.15 (P12)
- net Tile_28: now also U302.20 (P17); no longer U302.16 (P13)
- net Tile_29: now also U302.13 (P10); no longer U302.17 (P14)
- net Tile_30: now also U302.14 (P11); no longer U302.18 (P15)
- net Tile_31: now also U302.15 (P12); no longer U302.19 (P16)
- net Tile_32: now also U302.16 (P13); no longer U302.20 (P17)
- net Tile_41: now also U303.17 (P14); no longer U303.13 (P10)
- net Tile_42: now also U303.18 (P15); no longer U303.14 (P11)
- net Tile_43: now also U303.19 (P16); no longer U303.15 (P12)
- net Tile_44: now also U303.20 (P17); no longer U303.16 (P13)
- net Tile_45: now also U303.13 (P10); no longer U303.17 (P14)
- net Tile_46: now also U303.14 (P11); no longer U303.18 (P15)
- net Tile_47: now also U303.15 (P12); no longer U303.19 (P16)
- net Tile_48: now also U303.16 (P13); no longer U303.20 (P17)
- net Tile_57: now also U304.17 (P14); no longer U304.13 (P10)
- net Tile_58: now also U304.18 (P15); no longer U304.14 (P11)
- net Tile_59: now also U304.19 (P16); no longer U304.15 (P12)
- net Tile_60: now also U304.20 (P17); no longer U304.16 (P13)
- net Tile_61: now also U304.13 (P10); no longer U304.17 (P14)
- net Tile_62: now also U304.14 (P11); no longer U304.18 (P15)
- net Tile_63: now also U304.15 (P12); no longer U304.19 (P16)
- net Tile_64: now also U304.16 (P13); no longer U304.20 (P17)

Commit message: update schematic to include more components
Added SD card
Added IO expander for tactile buttons
Parts:
- added R305, R306, R307, R308, R309, R310, R311, R312, R313, R314, R315: (no value), symbol Device:R_Small
- added U305: (no value), symbol Interface_Expansion:TCA9535PWR
Connections:
- net 3V3: now also R305.1, R306.1, R307.1, R308.1, R309.1, R310.1, R311.1, R312.1, R313.1, R314.1, R315.1, U305.24 (VCC)
- net GND: now also U305.12 (GND), U305.2 (A1), U305.21 (A0)
- net ~{IO_INT}: now also U305.1 (~{INT})
- net ~{SCL_IOMUX}: now also U305.22 (SCL)
- net ~{SDA_IOMUX}: now also U305.23 (SDA)
- new net: R315.2, U305.3 (A2)
- new net B_DRAW: R313.2, U305.14 (P11)
- new net B_END: R311.2, U305.13 (P10)
- new net B_MOVE: R314.2, U305.15 (P12)
- new net MENU: R308.2, U305.5 (P01)
- new net SELECT: R310.2, U305.6 (P02)
- new net SET: R312.2, U305.7 (P03)
- new net START: R306.2, U305.4 (P00)
- new net W_DRAW: R307.2, U305.9 (P05)
- new net W_END: R305.2, U305.8 (P04)
- new net W_MOVE: R309.2, U305.10 (P06)
- no-connect marks 0 -> 6
Other:
- note added: "IO Expander for Hall Sensors"
- note added: "IO Expander for Tactile Buttons"
- note added: "Pull-Up Resistors for Tactile Buttons"
- moved on the sheet: R301, R302, R303, R304, U301, U302, U303, U304

Commit message: update PCB layout
Connections:
- net GND: no longer R304.2, U304.21 (A0)
- new net: R304.2, U304.21 (A0)
Changed lines of the file:
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@@
   (junction (at 205.74 34.29) (diameter 0) (color 0 0 0 0)
-  )
-  (junction (at 116.84 152.4) (diameter 0) (color 0 0 0 0)
   )
   (no_connect (at 247.65 139.7))
@@
     (stroke (width 0) (type default) (color 0 0 0 0))
   )
-  (wire (pts (xy 105.41 152.4) (xy 116.84 152.4))
-    (stroke (width 0) (type default) (color 0 0 0 0))
-  )
   (wire (pts (xy 243.84 34.29) (xy 240.03 34.29))
     (stroke (width 0) (type default) (color 0 0 0 0))
@@
     (stroke (width 0) (type default) (color 0 0 0 0))
   )
+  (wire (pts (xy 116.84 147.32) (xy 116.84 160.02))
+    (stroke (width 0) (type default) (color 0 0 0 0))
+  )
   (wire (pts (xy 35.56 152.4) (xy 35.56 160.02))
     (stroke (width 0) (type default) (color 0 0 0 0))
@@
     (stroke (width 0) (type default) (color 0 0 0 0))
   )
-  (wire (pts (xy 116.84 152.4) (xy 116.84 160.02))
-    (stroke (width 0) (type default) (color 0 0 0 0))
-  )
   (wire (pts (xy 77.47 152.4) (xy 74.93 152.4))
     (stroke (width 0) (type default) (color 0 0 0 0))
@@
     (stroke (width 0) (type default) (color 0 0 0 0))
   )
-  (wire (pts (xy 116.84 152.4) (xy 120.65 152.4))
+  (wire (pts (xy 105.41 152.4) (xy 120.65 152.4))
     (stroke (width 0) (type default) (color 0 0 0 0))
   )
@@
     (stroke (width 0) (type default) (color 0 0 0 0))
   )
-  (wire (pts (xy 116.84 147.32) (xy 116.84 152.4))
-    (stroke (width 0) (type default) (color 0 0 0 0))
-  )

Commit message: repurpose design with Nextion display
Parts:
- removed R306, R308, R310, R312: (no value), symbol Device:R_Small
- R301, R302, R303, R304, R315: value (none) -> 4K7; footprint (none) -> Resistor_SMD:R_0603_1608Metric
- R305, R307, R309, R311, R313, R314: value (none) -> 100K; footprint (none) -> Resistor_SMD:R_0603_1608Metric
- U301, U302, U303, U304, U305: value (none) -> PCA9535C; footprint (none) -> Package_SO:TSSOP-24_4.4x7.8mm_P0.65mm
Connections:
- net MENU: no longer names the net of U305.5 (P01)
- net SELECT: no longer names the net of U305.6 (P02)
- net SET: no longer names the net of U305.7 (P03)
- net START: no longer names the net of U305.4 (P00)
- no-connect marks 6 -> 10
Other:
- note added: "I2C addr 0x40"
- note added: "I2C addr 0x41"
- note added: "I2C addr 0x42"
- note added: "I2C addr 0x43"
- note added: "I2C addr 0x44"
- moved on the sheet: R305, R307, R309, R311, R313, R314

Commit message: add bypass caps
Parts:
- added C301, C302, C303, C304, C305: (no value), symbol Device:C_Small
- R301, R302, R303, R304, R315: value 4K7 -> (none); footprint Resistor_SMD:R_0603_1608Metric -> (none)
- R305, R307, R309, R311, R313, R314: value 100K -> (none); footprint Resistor_SMD:R_0603_1608Metric -> (none); LCSC (none) -> C25803
- U301, U302, U303, U304, U305: value PCA9535C -> (none); footprint Package_SO:TSSOP-24_4.4x7.8mm_P0.65mm -> (none)
Connections:
- net 3V3: now also C301.1, C302.1, C303.1, C304.1, C305.1
- net GND: now also C301.2, C302.2, C303.2, C304.2, C305.2
Other:
- note added: "By-Pass Caps for each IO Expander"
- moved on the sheet: R305, R307, R309, R311, R313, R314

Commit message: update pin assignments and footprint for hall sensors
Other:
- company: (none) -> Butler Electronics
- title: (none) -> Smart Chessboard - I/O Expander
Changed lines of the file:
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@@
 (kicad_sch (version 20211123) (generator eeschema)
   (paper "A4")
+  (title_block
+    (title "Smart Chessboard - I/O Expander")
+    (rev "A")
+    (company "Butler Electronics")
+    (comment 1 "Design by Joshua Butler, MD, MHI")
+  )
   (junction (at 115.57 72.39) (diameter 0) (color 0 0 0 0)
   )
