File: io_expander_sensor_switches.kicad_sch (KiCad schematic)
At the start: 21 parts

Commit message: add pull ups, bypass caps for SD card
Parts:
- C301, C302, C303, C304, C305: value (none) -> 100nF; footprint (none) -> Capacitor_SMD:C_0603_1608Metric
- R301, R302, R303, R304, R315: value (none) -> 4K7; footprint (none) -> Resistor_SMD:R_0603_1608Metric
- R305, R307, R309, R311, R313, R314: value (none) -> 100K; footprint (none) -> Resistor_SMD:R_0603_1608Metric
- U301, U302, U303, U304, U305: value (none) -> PCA9535C; footprint (none) -> Package_SO:TSSOP-24_4.4x7.8mm_P0.65mm
