File: hall_sensors.kicad_sch (KiCad schematic)
At the start: 192 parts

Commit message: update schematic with corrections
Connections:
- net Tile_55: now also R455.2, U455.2 (VOUT)
Changed lines of the file:
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@@
     )
   )
-  (global_label "Tile_55" (shape output) (at 349.25 245.11 0) (fields_autoplaced)
-    (effects (font (size 1.27 1.27)) (justify left))
-    (property "Intersheet References" "${INTERSHEET_REFS}" (id 0) (at 358.376 245.0306 0)
+  (global_label "Tile_55" (shape output) (at 349.25 246.38 0) (fields_autoplaced)
+    (effects (font (size 1.27 1.27)) (justify left))
+    (property "Intersheet References" "${INTERSHEET_REFS}" (id 0) (at 358.376 246.3006 0)
       (effects (font (size 1.27 1.27)) (justify left) hide)
     )
@@
       (effects (font (size 1.27 1.27)) hide)
     )
-    (property "Value" "" (id 1) (at 40.64 55.88 0)
-      (effects (font (size 1.27 1.27)) hide)
-    )
+    (property "Value" "GND" (id 1) (at 40.64 55.88 0)
+      (effects (font (size 1.27 1.27)) hide)
+    )

Commit message: repurpose design with Nextion display
Parts:
- C401, C402, C403, C404, C405, C406, C407, C408, C409, C410, C411, C412, C413, C414, C415, C416, C417, C418, C419, C420, C421, C422, C423, C424, C425, C426, C427, C428, C429, C430, C431, C432, C433, C434, C435, C436, C437, C438, C439, C440, C441, C442, C443, C444, C445, C446, C447, C448, C449, C450, C451, C452, C453, C454, C455, C456, C457, C458, C459, C460, C461, C462, C463, C464: value (none) -> 100nF; footprint (none) -> Capacitor_SMD:C_0603_1608Metric
- R401, R402, R403, R404, R405, R406, R407, R408, R409, R410, R411, R412, R413, R414, R415, R416, R417, R418, R419, R420, R421, R422, R423, R424, R425, R426, R427, R428, R429, R430, R431, R432, R433, R434, R435, R436, R437, R438, R439, R440, R441, R442, R443, R444, R445, R446, R447, R448, R449, R450, R451, R452, R453, R454, R455, R456, R457, R458, R459, R460, R461, R462, R463, R464: value (none) -> 2K7; footprint (none) -> Resistor_SMD:R_0603_1608Metric
- U401, U402, U403, U404, U405, U406, U407, U408, U409, U410, U411, U412, U413, U414, U415, U416, U417, U418, U419, U420, U421, U422, U423, U424, U425, U426, U427, U428, U429, U430, U431, U432, U433, U434, U435, U436, U437, U438, U439, U440, U441, U442, U443, U444, U445, U446, U447, U448, U449, U450, U451, U452, U453, U454, U455, U456, U457, U458, U459, U460, U461, U462, U463, U464: value (none) -> UHE4913; footprint (none) -> Package_TO_SOT_SMD:SOT-23

Commit message: add bypass caps
Parts:
- C401, C402, C403, C404, C405, C406, C407, C408, C409, C410, C411, C412, C413, C414, C415, C416, C417, C418, C419, C420, C421, C422, C423, C424, C425, C426, C427, C428, C429, C430, C431, C432, C433, C434, C435, C436, C437, C438, C439, C440, C441, C442, C443, C444, C445, C446, C447, C448, C449, C450, C451, C452, C453, C454, C455, C456, C457, C458, C459, C460, C461, C462, C463, C464: value 100nF -> (none); footprint Capacitor_SMD:C_0603_1608Metric -> (none)
- R401, R402, R403, R404, R405, R406, R407, R408, R409, R410, R411, R412, R413, R414, R415, R416, R417, R418, R419, R420, R421, R422, R423, R424, R425, R426, R427, R428, R429, R430, R431, R432, R433, R434, R435, R436, R437, R438, R439, R440, R441, R442, R443, R444, R445, R446, R447, R448, R449, R450, R451, R452, R453, R454, R455, R456, R457, R458, R459, R460, R461, R462, R463, R464: value 2K7 -> (none); footprint Resistor_SMD:R_0603_1608Metric -> (none)
- U401, U402, U403, U404, U405, U406, U407, U408, U409, U410, U411, U412, U413, U414, U415, U416, U417, U418, U419, U420, U421, U422, U423, U424, U425, U426, U427, U428, U429, U430, U431, U432, U433, U434, U435, U436, U437, U438, U439, U440, U441, U442, U443, U444, U445, U446, U447, U448, U449, U450, U451, U452, U453, U454, U455, U456, U457, U458, U459, U460, U461, U462, U463, U464: value UHE4913 -> (none); footprint Package_TO_SOT_SMD:SOT-23 -> (none)

Commit message: update pin assignments and footprint for hall sensors
Connections:
- net 3V3: now also U401.2 (VDD), U402.2 (VDD), U403.2 (VDD), U404.2 (VDD), U405.2 (VDD), U406.2 (VDD), U407.2 (VDD), U408.2 (VDD), U409.2 (VDD), U410.2 (VDD), U411.2 (VDD), U412.2 (VDD), U413.2 (VDD), U414.2 (VDD), U415.2 (VDD), U416.2 (VDD), U417.2 (VDD), U418.2 (VDD), U419.2 (VDD), U420.2 (VDD), U421.2 (VDD), U422.2 (VDD), U423.2 (VDD), U424.2 (VDD), U425.2 (VDD), U426.2 (VDD), U427.2 (VDD), U428.2 (VDD), U429.2 (VDD), U430.2 (VDD), U431.2 (VDD), U432.2 (VDD), U433.2 (VDD), U434.2 (VDD), U435.2 (VDD), U436.2 (VDD), U437.2 (VDD), U438.2 (VDD), U439.2 (VDD), U440.2 (VDD), U441.2 (VDD), U442.2 (VDD), U443.2 (VDD), U444.2 (VDD), U445.2 (VDD), U446.2 (VDD), U447.2 (VDD), U448.2 (VDD), U449.2 (VDD), U450.2 (VDD), U451.2 (VDD), U452.2 (VDD), U453.2 (VDD), U454.2 (VDD), U455.2 (VDD), U456.2 (VDD), U457.2 (VDD), U458.2 (VDD), U459.2 (VDD), U460.2 (VDD), U461.2 (VDD), U462.2 (VDD), U463.2 (VDD), U464.2 (VDD); no longer U401.1 (VDD), U402.1 (VDD), U403.1 (VDD), U404.1 (VDD), U405.1 (VDD), U406.1 (VDD), U407.1 (VDD), U408.1 (VDD), U409.1 (VDD), U410.1 (VDD), U411.1 (VDD), U412.1 (VDD), U413.1 (VDD), U414.1 (VDD), U415.1 (VDD), U416.1 (VDD), U417.1 (VDD), U418.1 (VDD), U419.1 (VDD), U420.1 (VDD), U421.1 (VDD), U422.1 (VDD), U423.1 (VDD), U424.1 (VDD), U425.1 (VDD), U426.1 (VDD), U427.1 (VDD), U428.1 (VDD), U429.1 (VDD), U430.1 (VDD), U431.1 (VDD), U432.1 (VDD), U433.1 (VDD), U434.1 (VDD), U435.1 (VDD), U436.1 (VDD), U437.1 (VDD), U438.1 (VDD), U439.1 (VDD), U440.1 (VDD), U441.1 (VDD), U442.1 (VDD), U443.1 (VDD), U444.1 (VDD), U445.1 (VDD), U446.1 (VDD), U447.1 (VDD), U448.1 (VDD), U449.1 (VDD), U450.1 (VDD), U451.1 (VDD), U452.1 (VDD), U453.1 (VDD), U454.1 (VDD), U455.1 (VDD), U456.1 (VDD), U457.1 (VDD), U458.1 (VDD), U459.1 (VDD), U460.1 (VDD), U461.1 (VDD), U462.1 (VDD), U463.1 (VDD), U464.1 (VDD)
- net Tile_01: now also U401.1 (VOUT); no longer U401.2 (VOUT)
- net Tile_02: now also U402.1 (VOUT); no longer U402.2 (VOUT)
- net Tile_03: now also U403.1 (VOUT); no longer U403.2 (VOUT)
- net Tile_04: now also U404.1 (VOUT); no longer U404.2 (VOUT)
- net Tile_05: now also U405.1 (VOUT); no longer U405.2 (VOUT)
- net Tile_06: now also U406.1 (VOUT); no longer U406.2 (VOUT)
- net Tile_07: now also U407.1 (VOUT); no longer U407.2 (VOUT)
- net Tile_08: now also U408.1 (VOUT); no longer U408.2 (VOUT)
- net Tile_09: now also U409.1 (VOUT); no longer U409.2 (VOUT)
- net Tile_10: now also U410.1 (VOUT); no longer U410.2 (VOUT)
- net Tile_11: now also U411.1 (VOUT); no longer U411.2 (VOUT)
- net Tile_12: now also U412.1 (VOUT); no longer U412.2 (VOUT)
- net Tile_13: now also U413.1 (VOUT); no longer U413.2 (VOUT)
- net Tile_14: now also U414.1 (VOUT); no longer U414.2 (VOUT)
- net Tile_15: now also U415.1 (VOUT); no longer U415.2 (VOUT)
- net Tile_16: now also U416.1 (VOUT); no longer U416.2 (VOUT)
- net Tile_17: now also U417.1 (VOUT); no longer U417.2 (VOUT)
- net Tile_18: now also U418.1 (VOUT); no longer U418.2 (VOUT)
- net Tile_19: now also U419.1 (VOUT); no longer U419.2 (VOUT)
- net Tile_20: now also U420.1 (VOUT); no longer U420.2 (VOUT)
- net Tile_21: now also U421.1 (VOUT); no longer U421.2 (VOUT)
- net Tile_22: now also U422.1 (VOUT); no longer U422.2 (VOUT)
- net Tile_23: now also U423.1 (VOUT); no longer U423.2 (VOUT)
- net Tile_24: now also U424.1 (VOUT); no longer U424.2 (VOUT)
- net Tile_25: now also U425.1 (VOUT); no longer U425.2 (VOUT)
- net Tile_26: now also U426.1 (VOUT); no longer U426.2 (VOUT)
- net Tile_27: now also U427.1 (VOUT); no longer U427.2 (VOUT)
- net Tile_28: now also U428.1 (VOUT); no longer U428.2 (VOUT)
- net Tile_29: now also U429.1 (VOUT); no longer U429.2 (VOUT)
- net Tile_30: now also U430.1 (VOUT); no longer U430.2 (VOUT)
- net Tile_31: now also U431.1 (VOUT); no longer U431.2 (VOUT)
- net Tile_32: now also U432.1 (VOUT); no longer U432.2 (VOUT)
- net Tile_33: now also U433.1 (VOUT); no longer U433.2 (VOUT)
- net Tile_34: now also U434.1 (VOUT); no longer U434.2 (VOUT)
- net Tile_35: now also U435.1 (VOUT); no longer U435.2 (VOUT)
- net Tile_36: now also U436.1 (VOUT); no longer U436.2 (VOUT)
- net Tile_37: now also U437.1 (VOUT); no longer U437.2 (VOUT)
- net Tile_38: now also U438.1 (VOUT); no longer U438.2 (VOUT)
- net Tile_39: now also U439.1 (VOUT); no longer U439.2 (VOUT)
- net Tile_40: now also U440.1 (VOUT); no longer U440.2 (VOUT)
- net Tile_41: now also U441.1 (VOUT); no longer U441.2 (VOUT)
- net Tile_42: now also U442.1 (VOUT); no longer U442.2 (VOUT)
- net Tile_43: now also U443.1 (VOUT); no longer U443.2 (VOUT)
- net Tile_44: now also U444.1 (VOUT); no longer U444.2 (VOUT)
- net Tile_45: now also U445.1 (VOUT); no longer U445.2 (VOUT)
- net Tile_46: now also U446.1 (VOUT); no longer U446.2 (VOUT)
- net Tile_47: now also U447.1 (VOUT); no longer U447.2 (VOUT)
- net Tile_48: now also U448.1 (VOUT); no longer U448.2 (VOUT)
- net Tile_49: now also U449.1 (VOUT); no longer U449.2 (VOUT)
- net Tile_50: now also U450.1 (VOUT); no longer U450.2 (VOUT)
- net Tile_51: now also U451.1 (VOUT); no longer U451.2 (VOUT)
- net Tile_52: now also U452.1 (VOUT); no longer U452.2 (VOUT)
- net Tile_53: now also U453.1 (VOUT); no longer U453.2 (VOUT)
- net Tile_54: now also U454.1 (VOUT); no longer U454.2 (VOUT)
- net Tile_55: now also U455.1 (VOUT); no longer U455.2 (VOUT)
- net Tile_56: now also U456.1 (VOUT); no longer U456.2 (VOUT)
- net Tile_57: now also U457.1 (VOUT); no longer U457.2 (VOUT)
- net Tile_58: now also U458.1 (VOUT); no longer U458.2 (VOUT)
- net Tile_59: now also U459.1 (VOUT); no longer U459.2 (VOUT)
- net Tile_60: now also U460.1 (VOUT); no longer U460.2 (VOUT)
- net Tile_61: now also U461.1 (VOUT); no longer U461.2 (VOUT)
- net Tile_62: now also U462.1 (VOUT); no longer U462.2 (VOUT)
- net Tile_63: now also U463.1 (VOUT); no longer U463.2 (VOUT)
- net Tile_64: now also U464.1 (VOUT); no longer U464.2 (VOUT)
Other:
- note added: "Note:"
- note added: "Pin assignments according to the UHE4913 datasheet: Pin 1 - Vout Pin 2 - Vdd Pin 3 - Ground But for SOT-23 footprint, the datasheet had pins 1 and 2 flipped. So the pin number on the symbol here on the schematic were flipped accordingly so that the pin assignment in the footprint matches the pin assignment in the datasheet eventhough the pin numbers were flipped."
- company: (none) -> Butler Electronics
- title: (none) -> Smart Chessboard - Hall Effect Sensors

Commit message: remove notes
Other:
- note removed: "Note:"
- note removed: "Pin assignments according to the UHE4913 datasheet: Pin 1 - Vout Pin 2 - Vdd Pin 3 - Ground But for SOT-23 footprint, the datasheet had pins 1 and 2 flipped. So the pin number on the symbol here on the schematic were flipped accordingly so that the pin assignment in the footprint matches the pin assignment in the datasheet eventhough the pin numbers were flipped."
Changed lines of the file:
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@@
-    (stroke (width 0) (type default) (color 0 0 0 0))
-  )
-  (polyline (pts (xy 33.02 295.91) (xy 33.02 336.55))
     (stroke (width 0) (type default) (color 0 0 0 0))
   )
@@
     (stroke (width 0) (type default) (color 0 0 0 0))
   )
-  (polyline (pts (xy 33.02 295.91) (xy 138.43 295.91))
-    (stroke (width 0) (type default) (color 0 0 0 0))
-  )
   (wire (pts (xy 322.58 201.93) (xy 330.2 201.93))
     (stroke (width 0) (type default) (color 0 0 0 0))
@@
     (stroke (width 0) (type default) (color 0 0 0 0))
   )
-  (polyline (pts (xy 138.43 295.91) (xy 138.43 336.55))
-    (stroke (width 0) (type default) (color 0 0 0 0))
-  )
   (wire (pts (xy 149.86 280.67) (xy 152.4 280.67))
     (stroke (width 0) (type default) (color 0 0 0 0))
@@
     (stroke (width 0) (type default) (color 0 0 0 0))
   )
-  (polyline (pts (xy 138.43 336.55) (xy 33.02 336.55))
-    (stroke (width 0) (type default) (color 0 0 0 0))
-  )
   (wire (pts (xy 322.58 175.26) (xy 322.58 167.64))
     (stroke (width 0) (type default) (color 0 0 0 0))
@@
     (stroke (width 0) (type default) (color 0 0 0 0))
   )
-  (text "Pin assignments according to the UHE4913 datasheet:\nPin 1 - Vout\nPin 2 - Vdd\nPin 3 - Ground\n\nBut for SOT-23 footprint, the datasheet had pins 1 and 2 flipped.\nSo the pin number on the symbol here on the schematic were\nflipped accordingly so that the pin assignment in the footprint\nmatches the pin assignment in the datasheet eventhough the pin\nnumbers were flipped. "
-    (at 34.29 335.28 0)
-    (effects (font (size 2 2) italic) (justify left bottom))
-  )
-  (text "Note:" (at 34.29 300.99 0)
-    (effects (font (size 3 3) (thickness 0.254) bold italic) (justify left bottom))
-  )
   (global_label "Tile_18" (shape output) (at 107.95 109.22 0) (fields_autoplaced)

Commit message: add pull ups, bypass caps for SD card
Parts:
- C401, C402, C403, C404, C405, C406, C407, C408, C409, C410, C411, C412, C413, C414, C415, C416, C417, C418, C419, C420, C421, C422, C423, C424, C425, C426, C427, C428, C429, C430, C431, C432, C433, C434, C435, C436, C437, C438, C439, C440, C441, C442, C443, C444, C445, C446, C447, C448, C449, C450, C451, C452, C453, C454, C455, C456, C457, C458, C459, C460, C461, C462, C463, C464: value (none) -> 100nF; footprint (none) -> Capacitor_SMD:C_0603_1608Metric
- R401, R402, R403, R404, R405, R406, R407, R408, R409, R410, R411, R412, R413, R414, R415, R416, R417, R418, R419, R420, R421, R422, R423, R424, R425, R426, R427, R428, R429, R430, R431, R432, R433, R434, R435, R436, R437, R438, R439, R440, R441, R442, R443, R444, R445, R446, R447, R448, R449, R450, R451, R452, R453, R454, R455, R456, R457, R458, R459, R460, R461, R462, R463, R464: value (none) -> 2K7; footprint (none) -> Resistor_SMD:R_0603_1608Metric
- U401, U402, U403, U404, U405, U406, U407, U408, U409, U410, U411, U412, U413, U414, U415, U416, U417, U418, U419, U420, U421, U422, U423, U424, U425, U426, U427, U428, U429, U430, U431, U432, U433, U434, U435, U436, U437, U438, U439, U440, U441, U442, U443, U444, U445, U446, U447, U448, U449, U450, U451, U452, U453, U454, U455, U456, U457, U458, U459, U460, U461, U462, U463, U464: value (none) -> UHE4913; footprint (none) -> User Custom Footprint:SOT-23-12_Flipped
