File: rgb_addr_led.kicad_sch (KiCad schematic)
At the start: 193 parts

Commit message: add level translator and fix OLED pin assignment
Parts:
- added C265, C266: (no value), symbol Device:C_Small
- added U201: (no value), symbol Logic_LevelTranslator:TXS0102DCU
- R213: LCSC C22775 -> C13167
Connections:
- net 5V: now also C266.1, U201.7 (VCCB)
- net GND: now also C265.1, C266.2, U201.2 (GND)
- net LED_IC: now also U201.5 (A1); no longer R213.1
- net at D201.4 (DIN), D202.6 (BIN): now also U201.8 (B1); no longer R213.2
- new net: R213.2, U201.6 (OE)
- new net 3V3: C265.2, R213.1, U201.3 (VCCA)
- no-connect marks 1 -> 3
Other:
- note added: "Logic Level Translator is needed as WS2813C V_{IH} is 0.7 * VDD = 3.5V. And the MCU only outputs at 3V3."
- note added: "NOTE:"
- moved on the sheet: C201, C202, C203, C204, C205, C206, C207, C208, C209, C210, C211, C212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

Commit message: repurpose design with Nextion display
Parts:
- C201, C202, C203, C204, C205, C206, C207, C208, C209, C210, C211, C212, C213, C214, C215, C216, C217, C218, C219, C220, C221, C222, C223, C224, C225, C226, C227, C228, C229, C230, C231, C232, C233, C234, C235, C236, C237, C238, C239, C240, C241, C242, C243, C244, C245, C246, C247, C248, C249, C250, C251, C252, C253, C254, C255, C256, C257, C258, C259, C260, C261, C262, C263, C264, C265, C266: value (none) -> 100nF; footprint (none) -> Capacitor_SMD:C_0603_1608Metric
- D201, D202, D203, D204, D205, D206, D207, D208, D209, D210, D211, D212, D213, D214, D215, D216, D217, D218, D219, D220, D221, D222, D223, D224, D225, D226, D227, D228, D229, D230, D231, D232, D233, D234, D235, D236, D237, D238, D239, D240, D241, D242, D243, D244, D245, D246, D247, D248, D249, D250, D251, D252, D253, D254, D255, D256, D257, D258, D259, D260, D261, D262, D263, D264: value (none) -> WS2813C; footprint (none) -> LED_SMD:LED_WS2812_PLCC6_5.0x5.0mm_P1.6mm
- R201, R202, R203, R204, R205, R206, R207, R208, R209, R210, R211, R212, R214, R215, R216, R217, R218, R219, R220, R221, R222, R223, R224, R225, R226, R227, R228, R229, R230, R231, R232, R233, R234, R235, R236, R237, R238, R239, R240, R241, R242, R243, R244, R245, R246, R247, R248, R249, R250, R251, R252, R253, R254, R255, R256, R257, R258, R259, R260, R261, R262, R263, R264, R265: value (none) -> 200; footprint (none) -> Resistor_SMD:R_0603_1608Metric
- R213: value (none) -> 100K; footprint (none) -> Resistor_SMD:R_0603_1608Metric
- U201: value (none) -> TXS0102DCU; footprint (none) -> Package_SO:VSSOP-8_2.3x2mm_P0.5mm

Commit message: add bypass caps
Parts:
- C201, C202, C203, C204, C205, C206, C207, C208, C209, C210, C211, C212, C213, C214, C215, C216, C217, C218, C219, C220, C221, C222, C223, C224, C225, C226, C227, C228, C229, C230, C231, C232, C233, C234, C235, C236, C237, C238, C239, C240, C241, C242, C243, C244, C245, C246, C247, C248, C249, C250, C251, C252, C253, C254, C255, C256, C257, C258, C259, C260, C261, C262, C263, C264, C265, C266: value 100nF -> (none); footprint Capacitor_SMD:C_0603_1608Metric -> (none)
- D201, D202, D203, D204, D205, D206, D207, D208, D209, D210, D211, D212, D213, D214, D215, D216, D217, D218, D219, D220, D221, D222, D223, D224, D225, D226, D227, D228, D229, D230, D231, D232, D233, D234, D235, D236, D237, D238, D239, D240, D241, D242, D243, D244, D245, D246, D247, D248, D249, D250, D251, D252, D253, D254, D255, D256, D257, D258, D259, D260, D261, D262, D263, D264: value WS2813C -> (none); footprint LED_SMD:LED_WS2812_PLCC6_5.0x5.0mm_P1.6mm -> (none)
- R201, R202, R203, R204, R205, R206, R207, R208, R209, R210, R211, R212, R214, R215, R216, R217, R218, R219, R220, R221, R222, R223, R224, R225, R226, R227, R228, R229, R230, R231, R232, R233, R234, R235, R236, R237, R238, R239, R240, R241, R242, R243, R244, R245, R246, R247, R248, R249, R250, R251, R252, R253, R254, R255, R256, R257, R258, R259, R260, R261, R262, R263, R264, R265: value 200 -> (none); footprint Resistor_SMD:R_0603_1608Metric -> (none)
- R213: value 100K -> (none); footprint Resistor_SMD:R_0603_1608Metric -> (none); LCSC C13167 -> C25803
- U201: value TXS0102DCU -> (none); footprint Package_SO:VSSOP-8_2.3x2mm_P0.5mm -> (none)
Other:
- note added: "By-pass Caps"
- moved on the sheet: C265, C266

Commit message: update pin assignments and footprint for hall sensors
Other:
- company: (none) -> Butler Electronics
- title: (none) -> Smart Chessboard - Addressable RGB LEDs
Changed lines of the file:
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@@
 (kicad_sch (version 20211123) (generator eeschema)
   (paper "A3")
+  (title_block
+    (title "Smart Chessboard - Addressable RGB LEDs")
+    (rev "A")
+    (company "Butler Electronics")
+    (comment 1 "Design by Joshua Butler, MD, MHI")
+  )
   (junction (at 163.83 214.63) (diameter 0) (color 0 0 0 0)
   )

Commit message: add pull ups, bypass caps for SD card
Parts:
- C201, C202, C203, C204, C205, C206, C207, C208, C209, C210, C211, C212, C213, C214, C215, C216, C217, C218, C219, C220, C221, C222, C223, C224, C225, C226, C227, C228, C229, C230, C231, C232, C233, C234, C235, C236, C237, C238, C239, C240, C241, C242, C243, C244, C245, C246, C247, C248, C249, C250, C251, C252, C253, C254, C255, C256, C257, C258, C259, C260, C261, C262, C263, C264, C265, C266: value (none) -> 100nF; footprint (none) -> Capacitor_SMD:C_0603_1608Metric
- D201, D202, D203, D204, D205, D206, D207, D208, D209, D210, D211, D212, D213, D214, D215, D216, D217, D218, D219, D220, D221, D222, D223, D224, D225, D226, D227, D228, D229, D230, D231, D232, D233, D234, D235, D236, D237, D238, D239, D240, D241, D242, D243, D244, D245, D246, D247, D248, D249, D250, D251, D252, D253, D254, D255, D256, D257, D258, D259, D260, D261, D262, D263, D264: value (none) -> WS2813C; footprint (none) -> LED_SMD:LED_WS2812_PLCC6_5.0x5.0mm_P1.6mm
- R201, R202, R203, R204, R205, R206, R207, R208, R209, R210, R211, R212, R214, R215, R216, R217, R218, R219, R220, R221, R222, R223, R224, R225, R226, R227, R228, R229, R230, R231, R232, R233, R234, R235, R236, R237, R238, R239, R240, R241, R242, R243, R244, R245, R246, R247, R248, R249, R250, R251, R252, R253, R254, R255, R256, R257, R258, R259, R260, R261, R262, R263, R264, R265: value (none) -> 200; footprint (none) -> Resistor_SMD:R_0603_1608Metric
- R213: value (none) -> 100K; footprint (none) -> Resistor_SMD:R_0603_1608Metric
- U201: value (none) -> TXS0102DCU; footprint (none) -> Package_SO:VSSOP-8_2.3x2mm_P0.5mm
